File: Phase B/Phase_B_Prototype.kicad_sch (KiCad schematic)
At the start: 48 parts, among them J1 USB_B_Mini, J3 AVR-ISP-6, J4 ESP_Conn, U1 CA56-12EWA, U2 74HC595, U3 ATmega32U4-A, U4 USBLC6-2SC6, U5 LP2985-3.3, Y1 16MHz

Commit message: Updated
Parts:
- C1, C10, C11, C12, C13, C14, C2, C3, C5, C6, C7, C8, C9: footprint Capacitor_SMD:C_0201_0603Metric -> Capacitor_SMD:C_0603_1608Metric
Connections:
- net Button_1: now also S1.B1 (NO_2); no longer S1.D1 (COM_2)
- net Button_2: now also S2.B1 (NO_2); no longer S2.D1 (COM_2)
Other:
- moved on the sheet: R1, R2
