File: Phase B/Phase_B_Prototype.kicad_pcb (KiCad board)
At the start: 2 copper layers, 99.1 x 71.1 mm, 48 parts, among them J1 USB_B_Mini, J3 AVR-ISP-6, J4 ESP_Conn, U1 CA56-12EWA, U2 74HC595, U3 ATmega32U4-A, U4 USBLC6-2SC6, U5 LP2985-3.3, Y1 16MHz

Commit message: Updated
Parts:
- moved J3 92.4 mm to (116.3, 118.9), turned to 180 degrees
- moved J1 64.7 mm to (121.4, 99.1), turned to -90 degrees
- moved D3 62.6 mm to (134.6, 89.3), turned to 90 degrees
- moved R14 59.4 mm to (138.6, 93.6)
- moved R15 54.9 mm to (138.5, 88.4)
- moved R16 54.9 mm to (138.5, 90.9)
- moved F2 54.8 mm to (132.2, 97.4)
- moved C11 50.9 mm to (144.3, 80.7), turned to 90 degrees
- moved C10 50.7 mm to (142.5, 80.7), turned to 90 degrees
- moved R13 49.4 mm to (144.9, 99.9), turned to 90 degrees
- moved U4 49.0 mm to (138.4, 84.5)
- moved S1 47.9 mm to (131.7, 116.6)
- moved C4 47.7 mm to (158.1, 82.0)
- moved R5 46.7 mm to (119.1, 58.7)
- moved R7 46.7 mm to (119.1, 64.6)
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Other:
- board size 99.1 x 71.1 mm -> 64.6 x 70 mm
- board text added: "Brian Lee 2023"
- board text added: "Embedded Systems Kitchen Timer"

Commit message: Updated
Parts:
- C1, C10, C11, C12, C13, C14, C2, C3, C5, C6, C7, C8, C9: footprint Capacitor_SMD:C_0201_0603Metric -> Capacitor_SMD:C_0603_1608Metric
- moved R4 41.6 mm to (166.3, 89.0), turned to 90 degrees
- moved D2 41.5 mm to (166.4, 85.3)
- moved R3 35.7 mm to (163.4, 89.0), turned to 90 degrees
- moved D1 35.5 mm to (163.4, 85.3)
- moved J4 26.8 mm to (155.2, 110.1), turned to 90 degrees
- moved C3 26.8 mm to (146.7, 108.2)
- moved J3 25.9 mm to (139.2, 106.9), turned to -90 degrees
- moved C6 22.4 mm to (140.5, 101.4), turned to 180 degrees
- moved C4 22.0 mm to (140.3, 95.0), turned to 180 degrees
- moved C1 21.1 mm to (145.7, 111.2), turned to -90 degrees
- moved C13 20.9 mm to (160.2, 105.8), turned to 90 degrees
- moved C5 20.9 mm to (140.4, 96.8), turned to 180 degrees
- moved C12 19.3 mm to (161.1, 102.7), turned to 180 degrees
- moved C10 19.2 mm to (140.5, 99.8), turned to 180 degrees
- moved S3 17.4 mm to (137.8, 112.4), turned to 180 degrees
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Connections:
- S1 pad B1: unconnected-(S1-NO_2-PadB1) -> Button_1
- S1 pad D1: Button_1 -> unconnected-(S1-COM_2-PadD1)
- S2 pad B1: unconnected-(S2-NO_2-PadB1) -> Button_2
- S2 pad D1: Button_2 -> unconnected-(S2-COM_2-PadD1)
Routing:
- net +5V: track 0.00 -> 160.0 mm, vias 0 -> 8
- net Dig3: track 0.00 -> 50.0 mm, vias 0 -> 2
- net Dig2: track 0.00 -> 47.2 mm, vias 0 -> 4
- net Buzzer: track 0.00 -> 45.6 mm
- net Dig1: track 0.00 -> 44.1 mm, vias 0 -> 2
- net Button_1: track 0.00 -> 42.6 mm, vias 0 -> 2
- net DS: track 0.00 -> 41.7 mm, vias 0 -> 2
- net ST_CP: track 0.00 -> 39.5 mm, vias 0 -> 2
- net Net-(U1-b): track 0.00 -> 35.0 mm
- net Net-(U1-f): track 0.00 -> 34.7 mm, vias 0 -> 4
- net Net-(U1-c): track 0.00 -> 34.1 mm
- net Net-(U1-g): track 0.00 -> 32.7 mm
- net a: track 0.00 -> 32.6 mm, vias 0 -> 2
- net Net-(U1-DPX): track 0.00 -> 29.3 mm, vias 0 -> 2
- net Button_2: track 0.00 -> 28.5 mm, vias 0 -> 2
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- added copper zone on B.Cu, net GND
Other:
- board size 64.6 x 70 mm -> 64.6 x 82.2 mm
- board text added: "Brian Lee April 2023"
- board text added: "Increment"
- board text added: "Start/Stop"
- board text removed: "Brian Lee 2023"

Commit message: Updated
Other:
- board text added: "Embedded Systems Kitchen Timer Version 1"
- board text removed: "Embedded Systems Kitchen Timer"
Changed lines of the file:
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@@
   (gr_rect (start 112.32 55.88) (end 176.88 138.06)
     (stroke (width 0.15) (type default)) (fill none) (layer "Edge.Cuts"))
-  (gr_text "Embedded Systems\nKitchen Timer" (at 175.7 59.9) (layer "B.SilkS")
+  (gr_text "Embedded Systems\nKitchen Timer\nVersion 1" (at 175.7 61.41) (layer "B.SilkS")
     (effects (font (size 1 1) (thickness 0.15)) (justify left bottom mirror))
   )
